Commit message: added workspace box

File: visualizer/6dof/urdf/6dof.urdf (robot description, URDF)
Before this commit: robot GEN3_LITE_6DOF_WITH_GRIPPER, 13 links, 12 joints
Links:
- added link WORKSPACE_INDICATOR; visual box size=0.6 0.6 0.6
Joints:
- added joint workspace_joint: type fixed, parent BASE, child WORKSPACE_INDICATOR, origin xyz=0.4 0.0 0.3 rpy=0 0 0
- joint J0: origin xyz=0 0 0.12825 rpy=0 0 0 -> xyz=0 0 0.12825 rpy=0 0 -1.57

File: visualizer/7dof/urdf/7dof.urdf (robot description, URDF)
Before this commit: robot GEN3_7DOF_WITH_EPICK, 11 links, 10 joints
Links:
- added link WORKSPACE_INDICATOR; visual box size=0.6 0.6 0.6
Joints:
- added joint workspace_joint: type fixed, parent base_link, child WORKSPACE_INDICATOR, origin xyz=0.4 0.0 0.3 rpy=0 0 0
