Commit message: added gripper and fixed simulator problem

File: visualizer/7dof/urdf/7dof_suction.urdf (robot description, URDF)
Before this commit: robot GEN3_7DOF_WITH_GRIPPER, 10 links, 9 joints
Links:
- added link epick_end_effector, mass 0.0001; visual cylinder length=0.01 radius=0.0225
- added link robotiq_epick_base_link, mass 0.745; collision cylinder length=0.13 radius=0.044; visual cylinder length=0.03 radius=0.006
Joints:
- added joint arm_to_epick: type fixed, parent EndEffector_Link, child robotiq_epick_base_link, origin xyz=0 0 0 rpy=0 0 0
- added joint epick_end_effector_joint: type fixed, parent robotiq_epick_base_link, child epick_end_effector, origin xyz=0 0 0.13 rpy=0 0 0
